Commit message: chore: rename px4_roscon_25 package to px4_roscon_workshop
Signed-off-by: Beniamino Pozzan <beniamino.pozzan@gmail.com>

File: px4_roscon_workshop/px4_roscon_workshop/urdf/x500.urdf (robot description, URDF)
Before this commit: robot x500, 5 links, 4 joints
Links:
- link base_link: geometry visual mesh filename=package://px4_roscon_workshop/meshes/5010Base.dae; visual mesh filename=package://px4_roscon_workshop/meshes/5010Base.dae
- link motor_0: geometry visual mesh filename=package://px4_roscon_workshop/meshes/5010Bell.dae
- link motor_1: geometry visual mesh filename=package://px4_roscon_workshop/meshes/5010Bell.dae
- link motor_2: geometry visual mesh filename=package://px4_roscon_workshop/meshes/5010Bell.dae
- link motor_3: geometry visual mesh filename=package://px4_roscon_workshop/meshes/5010Bell.dae
